File: Boost PCB.kicad_pcb (KiCad board)
At the start: 2 copper layers, 25 x 51 mm, 2 parts, among them J3 Conn_01x03_Pin, U1 BoostConverter

Commit message: Finished Boost PCB
Other:
- board text added: "HIGH SIDE (48V)"
- board text added: "LOW SIDE (12V)"
Changed lines of the file:
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@@
 		)
 		(embedded_fonts no)
+		(model "${KIPRJMOD}/XL6009_pin.stp"
+			(offset
+				(xyz 3 0 2.5)
+			)
+			(scale
+				(xyz 1 1 1)
+			)
+			(rotate
+				(xyz -90 -0 -0)
+			)
+		)
 	)
 	(footprint "Connector_JST:JST_XH_B3B-XH-A_1x03_P2.50mm_Vertical"
@@
 		(end 61.15 74.5)
 		(stroke
-			(width 0)
+			(width 0.1)
 			(type default)
 		)
@@
 		(end 36.15 74.5)
 		(stroke
-			(width 0)
+			(width 0.1)
 			(type default)
 		)
@@
 		(end 61.15 125.5)
 		(stroke
-			(width 0)
+			(width 0.1)
 			(type default)
 		)
@@
 		(end 61.15 74.5)
 		(stroke
-			(width 0)
+			(width 0.1)
 			(type default)
 		)
 		(layer "Edge.Cuts")
+	)
+	(gr_text "HIGH SIDE (48V)\n"
+		(at 39.1 80.21 0)
+		(layer "F.SilkS")
+		(effects
+			(font
+				(size 1.5 1.5)
+				(thickness 0.3)
+				(bold yes)
+			)
+			(justify left bottom)
+		)
+	)
+	(gr_text "LOW SIDE (12V)\n"
+		(at 57.6 119.71 180)
+		(layer "F.SilkS")
+		(effects
+			(font
+				(size 1.5 1.5)
+				(thickness 0.3)
+				(bold yes)
+			)
+			(justify left bottom)
+		)
 	)
 	(segment
@@
 	)
 	(segment
+		(start 51.57 84.52)
+		(end 51.57 115.65)
+		(width 2)
+		(layer "B.Cu")
+		(net "GND")
+	)
+	(segment
+		(start 48.65 87.31)
+		(end 43.525 87.31)
+		(width 2)
+		(layer "B.Cu")
+		(net "GND")
+	)
+	(segment
+		(start 51.57 115.65)
+		(end 58.94 123.02)
+		(width 2)
+		(layer "B.Cu")
+		(net "GND")
+	)
+	(segment
+		(start 51.505 84.455)
+		(end 51.57 84.52)
+		(width 2)
+		(layer "B.Cu")
+		(net "GND")
+	)
+	(segment
+		(start 58.94 77.02)
+		(end 51.505 84.455)
+		(width 2)
+		(layer "B.Cu")
+		(net "GND")
+	)
+	(segment
+		(start 51.505 84.455)
+		(end 48.65 87.31)
+		(width 2)
+		(layer "B.Cu")
+		(net "GND")
+	)
+	(segment
 		(start 40.8 89.81)
 		(end 43.525 89.81)
@@
 		(net "48V")
 	)
-	(segment
-		(start 51.57 84.52)
-		(end 51.57 115.65)
-		(width 2)
-		(layer "B.Cu")
-		(net "GND")
-	)
-	(segment
-		(start 48.65 87.31)
-		(end 43.525 87.31)
-		(width 2)
-		(layer "B.Cu")
-		(net "GND")
-	)
-	(segment
-		(start 51.57 115.65)
-		(end 58.94 123.02)
-		(width 2)
-		(layer "B.Cu")
-		(net "GND")
-	)
-	(segment
-		(start 51.505 84.455)
-		(end 51.57 84.52)
-		(width 2)
-		(layer "B.Cu")
-		(net "GND")
-	)
-	(segment
-		(start 58.94 77.02)
-		(end 51.505 84.455)
-		(width 2)
-		(layer "B.Cu")
-		(net "GND")
-	)
-	(segment
-		(start 51.505 84.455)
-		(end 48.65 87.31)
-		(width 2)
-		(layer "B.Cu")
-		(net "GND")
-	)
 	(zone

Commit message: Moved JST
Parts:
- moved J3 6.02 mm to (47.1, 80.0)
Routing:
- net 12V: track 51.6 -> 49.6 mm
- net GND: track 61.3 -> 59.6 mm
- net 48V: track 16.5 -> 15.2 mm
Changed lines of the file:
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@@
 	(footprint "Connector_JST:JST_XH_B3B-XH-A_1x03_P2.50mm_Vertical"
 		(layer "B.Cu")
-		(at 43.525 84.81 -90)
+		(at 47.15 80 -90)
 		(descr "JST XH series connector, B3B-XH-A (http://www.jst-mfg.com/product/pdf/eng/eXH.pdf)")
 		(tags "connector JST XH vertical")
@@
 	)
 	(segment
+		(start 48.125 80)
+		(end 47.15 80)
+		(width 2)
+		(layer "F.Cu")
+		(net "12V")
+	)
+	(segment
 		(start 50.07 111.39)
 		(end 38.44 123.02)
@@
 	)
 	(segment
-		(start 44.935 83.4)
-		(end 50.07 83.4)
+		(start 50.07 86.73)
+		(end 50.07 81.945)
 		(width 2)
 		(layer "F.Cu")
@@
 	)
 	(segment
-		(start 43.525 84.81)
-		(end 44.935 83.4)
+		(start 50.07 86.73)
+		(end 50.07 111.39)
 		(width 2)
 		(layer "F.Cu")
@@
 	)
 	(segment
-		(start 50.07 83.4)
-		(end 50.07 111.39)
+		(start 50.07 81.945)
+		(end 48.125 80)
 		(width 2)
 		(layer "F.Cu")
@@
 	)
 	(segment
+		(start 54.24 81.72)
+		(end 53.46 82.5)
+		(width 2)
+		(layer "B.Cu")
+		(net "GND")
+	)
+	(segment
 		(start 51.57 84.52)
 		(end 51.57 115.65)
@@
 	)
 	(segment
-		(start 48.65 87.31)
-		(end 43.525 87.31)
+		(start 54.24 81.72)
+		(end 51.505 84.455)
 		(width 2)
 		(layer "B.Cu")
@@
 	)
 	(segment
+		(start 53.46 82.5)
+		(end 47.15 82.5)
+		(width 2)
+		(layer "B.Cu")
+		(net "GND")
+	)
+	(segment
 		(start 58.94 77.02)
-		(end 51.505 84.455)
-		(width 2)
-		(layer "B.Cu")
-		(net "GND")
-	)
-	(segment
-		(start 51.505 84.455)
-		(end 48.65 87.31)
-		(width 2)
-		(layer "B.Cu")
-		(net "GND")
-	)
-	(segment
-		(start 40.8 89.81)
-		(end 43.525 89.81)
+		(end 54.24 81.72)
+		(width 2)
+		(layer "B.Cu")
+		(net "GND")
+	)
+	(segment
+		(start 38.44 77.02)
+		(end 38.44 82.43)
 		(width 2)
 		(layer "B.Cu")
@@
 	)
 	(segment
-		(start 38.44 77.02)
-		(end 38.44 87.45)
+		(start 41.01 85)
+		(end 47.15 85)
 		(width 2)
 		(layer "B.Cu")
@@
 	)
 	(segment
-		(start 38.44 87.45)
-		(end 40.8 89.81)
-		(width 2)
-		(layer "B.Cu")
+		(start 38.44 82.43)
+		(end 41.01 85)
+		(width 2)
+		(layer "B.Cu")
